File: Circuit Design/dc_controller/dc_controller.kicad_sch (KiCad schematic)
At the start: 46 parts, among them J1 Screw_Terminal_01x08, M1 Motor_DC, Q1 IRFB4110PBF NMOS, Q11 IRFB4110PBF NMOS, Q12 IRFB4110PBF NMOS, Q2 IRFB4110PBF NMOS, Q3 IRFB4110PBF NMOS, Q4 IRFB4110PBF NMOS, Q5 IRFB4110PBF NMOS, Q6 IRFB4110PBF NMOS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

Commit message: Update
Parts:
- R1, R2, R5, R6: value 22 -> 4.7
